Commit message: Port to ROS2 jazzy.

File: terry/config/robot_hardware_description.urdf (robot description, URDF)
Before this commit: robot terry, 0 links, 0 joints
Links:
- added link base_link
- added link front_wheel
- added link left_wheel
- added link right_wheel
Joints:
- added joint PORT_A: type continuous, parent base_link, child right_wheel
- added joint PORT_B: type continuous, parent base_link, child left_wheel
- added joint PORT_D: type continuous, parent base_link, child front_wheel
